Commit message: FIXXING:ロボットモデル修正中

File: happymimi_description/robots/happymimi.urdf.xacro (robot description, xacro)
@@ -1,3 +1,3 @@
-<?xml version="1.0" encoding="utf-8"?>
+<?xml version="1.0"?>
 <robot name="happymimiGen3" xmlns:xacro="http://ros.org/wiki/xacro">
   <xacro:include filename="$(find happymimi_description)/urdf/body/body.urdf.xacro"/>

File: happymimi_description/robots/vhappymimi.urdf.xacro (robot description, xacro)
@@ -28,9 +28,9 @@
   <!-- Front LRF Upper-->
   <!-- <xacro:lrf_v0 prefix="front" parent="base_link">
-  	<origin xyz="0.099 0 0.2155"  rpy="${M_PI} 0 0" />
+  <origin xyz="0.099 0 0.2155"  rpy="${M_PI} 0 0" />
   </xacro:lrf_v0> -->
   <!-- Rear LRF -->
   <!-- xacro:lrf_v0 prefix="rear" parent="base_link">
-  	<origin xyz="-0.289 0 0.1015"  rpy="0 0 ${M_PI}" />
+  <origin xyz="-0.289 0 0.1015"  rpy="0 0 ${M_PI}" />
   </xacro:lrf_v0 -->
   <!-- <link name="lrf_link"/> -->
@@ -72,10 +72,6 @@
   <xacro:wheel_gazebo_v0 prefix="left"/>
   <!-- LRF -->
-  <xacro:lrf_gazebo_v0 prefix="front"
-					   min_rad="-1.57" max_rad="1.57"
-					   min_range="0.06" max_range="4.0"/>
-  <!-- xacro:lrf_gazebo_v0 prefix="rear"
-					   min_rad="-1.57" max_rad="1.57"
-					   min_range="0.06" max_range="4.0"/ -->
+  <xacro:lrf_gazebo_v0 prefix="front" min_rad="-1.57" max_rad="1.57" min_range="0.06" max_range="4.0"/>
+  <!-- xacro:lrf_gazebo_v0 prefix="rear" min_rad="-1.57" max_rad="1.57" min_range="0.06" max_range="4.0"/ -->
   <!-- Realsense Gazebo Plugin -->
     <xacro:gazebo_d435 camera_name="realsense" reference_link="$realsense_link" topics_ns="camera" depth_optical_frame="realsense_depth_optical_frame" color_optical_frame="realsense_color_optical_frame" infrared1_optical_frame="realsense_left_ir_optical_frame" infrared2_optical_frame="realsense_right_ir_optical_frame"/>

File: happymimi_description/urdf/camera/d435.gazebo.xacro (robot description, xacro)
@@ -116,25 +116,25 @@
     <!--     <robotNamespace>/vhappymimi</robotNamespace> -->
     <!--     <prefix>${camera_name}</prefix> -->
-    <!--   	<depthUpdateRate>60.0</depthUpdateRate> -->
-    <!--   	<colorUpdateRate>60.0</colorUpdateRate> -->
-    <!--   	<infraredUpdateRate>60.0</infraredUpdateRate> -->
-    <!--   	<depthTopicName>depth/image_raw</depthTopicName> -->
-    <!--   	<depthCameraInfoTopicName>depth/camera_info</depthCameraInfoTopicName> -->
-    <!--   	<colorTopicName>color/image_raw</colorTopicName> -->
-    <!--   	<colorCameraInfoTopicName>color/camera_info</colorCameraInfoTopicName> -->
-    <!--   	<infrared1TopicName>infra1/image_raw</infrared1TopicName> -->
-    <!--   	<infrared1CameraInfoTopicName>infra1/camera_info</infrared1CameraInfoTopicName> -->
-    <!--   	<infrared2TopicName>infra2/image_raw</infrared2TopicName> -->
-    <!--   	<infrared2CameraInfoTopicName>infra2/camera_info</infrared2CameraInfoTopicName> -->
-    <!--   	<colorOpticalframeName>${color_optical_frame}</colorOpticalframeName> -->
-    <!--   	<depthOpticalframeName>${depth_optical_frame}</depthOpticalframeName> -->
-    <!--   	<infrared1OpticalframeName>${infrared1_optical_frame}</infrared1OpticalframeName> -->
-    <!--   	<infrared2OpticalframeName>${infrared2_optical_frame}</infrared2OpticalframeName> -->
-    <!--   	<rangeMinDepth>0.2</rangeMinDepth> -->
-    <!--   	<rangeMaxDepth>10.0</rangeMaxDepth> -->
-    <!--   	<pointCloud>false</pointCloud> -->
-    <!--   	<pointCloudTopicName>depth/points</pointCloudTopicName> -->
-    <!--   	<pointCloudCutoff>0.5</pointCloudCutoff> -->
-    <!--   </plugin> -->
+    <!--<depthUpdateRate>60.0</depthUpdateRate> -->
+    <!--<colorUpdateRate>60.0</colorUpdateRate> -->
+    <!--<infraredUpdateRate>60.0</infraredUpdateRate> -->
+    <!--<depthTopicName>depth/image_raw</depthTopicName> -->
+    <!--<depthCameraInfoTopicName>depth/camera_info</depthCameraInfoTopicName> -->
+    <!--<colorTopicName>color/image_raw</colorTopicName> -->
+    <!--<colorCameraInfoTopicName>color/camera_info</colorCameraInfoTopicName> -->
+    <!--<infrared1TopicName>infra1/image_raw</infrared1TopicName> -->
+    <!--<infrared1CameraInfoTopicName>infra1/camera_info</infrared1CameraInfoTopicName> -->
+    <!--<infrared2TopicName>infra2/image_raw</infrared2TopicName> -->
+    <!--<infrared2CameraInfoTopicName>infra2/camera_info</infrared2CameraInfoTopicName> -->
+    <!--<colorOpticalframeName>${color_optical_frame}</colorOpticalframeName> -->
+    <!--<depthOpticalframeName>${depth_optical_frame}</depthOpticalframeName> -->
+    <!--<infrared1OpticalframeName>${infrared1_optical_frame}</infrared1OpticalframeName> -->
+    <!--<infrared2OpticalframeName>${infrared2_optical_frame}</infrared2OpticalframeName> -->
+    <!--<rangeMinDepth>0.2</rangeMinDepth> -->
+    <!--<rangeMaxDepth>10.0</rangeMaxDepth> -->
+    <!--<pointCloud>false</pointCloud> -->
+    <!--<pointCloudTopicName>depth/points</pointCloudTopicName> -->
+    <!--<pointCloudCutoff>0.5</pointCloudCutoff> -->
+    <!--</plugin> -->
     <!-- </gazebo> -->
   </xacro:macro>
